File: hw/arm.sch (KiCad schematic (older format))
At the start: 12 parts, among them J4 SWD_01X04, U5 STM32F405RGTx

Commit message: updated schematic
Parts:
- added J3: UART_01X03, Connector_PinHeader_2.54mm:PinHeader_1x03_P2.54mm_Vertical, symbol KLIB_Connector_Prog:UART_01X03
- C10, C11, C12, C13, C14, C15, C16, C17: footprint (none) -> Capacitor_SMD:C_0805_2012Metric
- R11, R12: footprint (none) -> Resistor_SMD:R_0805_2012Metric
- U5: footprint LQFP64 -> Package_QFP:TQFP-64_10x10mm_P0.5mm
Connections:
- net DEBUG_UART_RX: now also J3.2 (RX)
- net DEBUG_UART_TX: now also J3.3 (TX)
- net GND: now also J3.1 (GND)
Changed lines of the file:
@@
 F 0 "U5" H 1650 5850 50  0000 L CNN
 F 1 "STM32F405RGTx" H 1650 5750 50  0000 L CNN
-F 2 "LQFP64" H 10050 5625 50  0001 R TNN
+F 2 "Package_QFP:TQFP-64_10x10mm_P0.5mm" H 10050 5625 50  0001 R TNN
 F 3 "http://www.st.com/st-web-ui/static/active/en/resource/technical/document/datasheet/DM00037051.pdf" H 5850 3750 50  0001 C CNN
 	1    5850 3750
@@
 $EndComp
 $Comp
-L KLIB_Power:+3V3 #PWR038
+L KLIB_Power:+3V3 #PWR037
 U 1 1 5ACE8468
 P 5850 1650
-F 0 "#PWR038" H 5850 1350 50  0001 C CNN
+F 0 "#PWR037" H 5850 1350 50  0001 C CNN
 F 1 "+3V3" H 5855 1823 50  0000 C CNN
 F 2 "" H 5850 1650 50  0001 C CNN
@@
 	5950 1700 6050 1700
 $Comp
-L KLIB_Power:GND #PWR039
+L KLIB_Power:GND #PWR038
 U 1 1 5ACE8945
 P 5850 5850
-F 0 "#PWR039" H 5850 5650 50  0001 C CNN
+F 0 "#PWR038" H 5850 5650 50  0001 C CNN
 F 1 "GND" H 5855 5677 50  0000 C CNN
 F 2 "" H 5850 5850 50  0001 C CNN
@@
 F 0 "R12" H 1170 1996 50  0000 L CNN
 F 1 "10k" H 1170 1905 50  0000 L CNN
-F 2 "" V 1030 1950 50  0001 C CNN
+F 2 "Resistor_SMD:R_0805_2012Metric" V 1030 1950 50  0001 C CNN
 F 3 "~" H 1100 1950 50  0001 C CNN
 	1    1100 1950
@@
 F 0 "R11" H 820 1996 50  0000 L CNN
 F 1 "10k" H 820 1905 50  0000 L CNN
-F 2 "" V 680 1950 50  0001 C CNN
+F 2 "Resistor_SMD:R_0805_2012Metric" V 680 1950 50  0001 C CNN
 F 3 "~" H 750 1950 50  0001 C CNN
 	1    750  1950
@@
 $EndComp
 $Comp
-L KLIB_Power:GND #PWR032
+L KLIB_Power:GND #PWR031
 U 1 1 5ACE95CC
 P 750 1700
-F 0 "#PWR032" H 750 1500 50  0001 C CNN
+F 0 "#PWR031" H 750 1500 50  0001 C CNN
 F 1 "GND" H 755 1527 50  0000 C CNN
 F 2 "" H 750 1700 50  0001 C CNN
@@
 $EndComp
 $Comp
-L KLIB_Power:+3V3 #PWR034
+L KLIB_Power:+3V3 #PWR033
 U 1 1 5ACE967B
 P 1100 1700
-F 0 "#PWR034" H 1100 1400 50  0001 C CNN
+F 0 "#PWR033" H 1100 1400 50  0001 C CNN
 F 1 "+3V3" H 1105 1873 50  0000 C CNN
 F 2 "" H 1100 1700 50  0001 C CNN
@@
 Text HLabel 10400 3350 2    50   Output ~ 0
 USB_UART_RTS
-Wire Wire Line
-	10150 4850 10400 4850
-Wire Wire Line
-	10150 4950 10400 4950
-Text HLabel 10400 4850 2    50   Output ~ 0
-DEBUG_UART_TX
-Text HLabel 10400 4950 2    50   Input ~ 0
-DEBUG_UART_RX
 Wire Wire Line
 	10150 2550 10400 2550
@@
 	5450 7100 5000 7100
 $Comp
-L KLIB_Power:GND #PWR037
+L KLIB_Power:GND #PWR036
 U 1 1 5ACFAB32
 P 5450 7200
-F 0 "#PWR037" H 5450 7000 50  0001 C CNN
+F 0 "#PWR036" H 5450 7000 50  0001 C CNN
 F 1 "GND" H 5455 7027 50  0000 C CNN
 F 2 "" H 5450 7200 50  0001 C CNN
@@
 F 0 "C10" H 865 2996 50  0000 L CNN
 F 1 "100n" H 865 2905 50  0000 L CNN
-F 2 "" H 788 2800 50  0001 C CNN
+F 2 "Capacitor_SMD:C_0805_2012Metric" H 788 2800 50  0001 C CNN
 F 3 "~" H 750 2950 50  0001 C CNN
 	1    750  2950
@@
 F 0 "C11" H 1365 2996 50  0000 L CNN
 F 1 "100n" H 1365 2905 50  0000 L CNN
-F 2 "" H 1288 2800 50  0001 C CNN
+F 2 "Capacitor_SMD:C_0805_2012Metric" H 1288 2800 50  0001 C CNN
 F 3 "~" H 1250 2950 50  0001 C CNN
 	1    1250 2950
@@
 $EndComp
 $Comp
-L KLIB_Power:GND #PWR035
+L KLIB_Power:GND #PWR034
 U 1 1 5AD22D21
 P 1250 3100
-F 0 "#PWR035" H 1250 2900 50  0001 C CNN
+F 0 "#PWR034" H 1250 2900 50  0001 C CNN
 F 1 "GND" H 1255 2927 50  0000 C CNN
 F 2 "" H 1250 3100 50  0001 C CNN
@@
 $EndComp
 $Comp
-L KLIB_Power:GND #PWR033
+L KLIB_Power:GND #PWR032
 U 1 1 5AD22D74
 P 750 3100
-F 0 "#PWR033" H 750 2900 50  0001 C CNN
+F 0 "#PWR032" H 750 2900 50  0001 C CNN
 F 1 "GND" H 755 2927 50  0000 C CNN
 F 2 "" H 750 3100 50  0001 C CNN
@@
 F 0 "C13" H 7865 1196 50  0000 L CNN
 F 1 "100n" H 7865 1105 50  0000 L CNN
-F 2 "" H 7788 1000 50  0001 C CNN
+F 2 "Capacitor_SMD:C_0805_2012Metric" H 7788 1000 50  0001 C CNN
 F 3 "~" H 7750 1150 50  0001 C CNN
 	1    7750 1150
@@
 F 0 "C14" H 8315 1196 50  0000 L CNN
 F 1 "100n" H 8315 1105 50  0000 L CNN
-F 2 "" H 8238 1000 50  0001 C CNN
+F 2 "Capacitor_SMD:C_0805_2012Metric" H 8238 1000 50  0001 C CNN
 F 3 "~" H 8200 1150 50  0001 C CNN
 	1    8200 1150
@@
 F 0 "C15" H 8765 1196 50  0000 L CNN
 F 1 "100n" H 8765 1105 50  0000 L CNN
-F 2 "" H 8688 1000 50  0001 C CNN
+F 2 "Capacitor_SMD:C_0805_2012Metric" H 8688 1000 50  0001 C CNN
 F 3 "~" H 8650 1150 50  0001 C CNN
 	1    8650 1150
@@
 F 0 "C16" H 9215 1196 50  0000 L CNN
 F 1 "100n" H 9215 1105 50  0000 L CNN
-F 2 "" H 9138 1000 50  0001 C CNN
+F 2 "Capacitor_SMD:C_0805_2012Metric" H 9138 1000 50  0001 C CNN
 F 3 "~" H 9100 1150 50  0001 C CNN
 	1    9100 1150
@@
 F 0 "C17" H 9665 1196 50  0000 L CNN
 F 1 "100n" H 9665 1105 50  0000 L CNN
-F 2 "" H 9588 1000 50  0001 C CNN
+F 2 "Capacitor_SMD:C_0805_2012Metric" H 9588 1000 50  0001 C CNN
 F 3 "~" H 9550 1150 50  0001 C CNN
 	1    9550 1150
@@
 F 0 "C12" H 7415 1196 50  0000 L CNN
 F 1 "100n" H 7415 1105 50  0000 L CNN
-F 2 "" H 7338 1000 50  0001 C CNN
+F 2 "Capacitor_SMD:C_0805_2012Metric" H 7338 1000 50  0001 C CNN
 F 3 "~" H 7300 1150 50  0001 C CNN
 	1    7300 1150
@@
 	9550 1000 9550 950
 $Comp
-L KLIB_Power:+3V3 #PWR040
+L KLIB_Power:+3V3 #PWR039
 U 1 1 5AD26399
 P 8450 900
-F 0 "#PWR040" H 8450 600 50  0001 C CNN
+F 0 "#PWR039" H 8450 600 50  0001 C CNN
 F 1 "+3V3" H 8455 1073 50  0000 C CNN
 F 2 "" H 8450 900 50  0001 C CNN
@@
 $EndComp
 $Comp
-L KLIB_Power:GND #PWR041
+L KLIB_Power:GND #PWR040
 U 1 1 5AD2639F
 P 8450 1400
-F 0 "#PWR041" H 8450 1200 50  0001 C CNN
+F 0 "#PWR040" H 8450 1200 50  0001 C CNN
 F 1 "GND" H 8455 1227 50  0000 C CNN
 F 2 "" H 8450 1400 50  0001 C CNN
@@
 LED[7..0]
 $Comp
-L KLIB_Power:PWR_FLAG #FLG0101
+L KLIB_Power:PWR_FLAG #FLG01
 U 1 1 5AE70DE3
 P 750 2600
-F 0 "#FLG0101" H 750 2675 50  0001 C CNN
+F 0 "#FLG01" H 750 2675 50  0001 C CNN
 F 1 "PWR_FLAG" H 750 2774 50  0000 C CNN
 F 2 "" H 750 2600 50  0001 C CNN
@@
 $EndComp
 $Comp
-L KLIB_Power:PWR_FLAG #FLG0102
+L KLIB_Power:PWR_FLAG #FLG02
 U 1 1 5AE70EFD
 P 1250 2600
-F 0 "#FLG0102" H 1250 2675 50  0001 C CNN
+F 0 "#FLG02" H 1250 2675 50  0001 C CNN
 F 1 "PWR_FLAG" H 1250 2774 50  0000 C CNN
 F 2 "" H 1250 2600 50  0001 C CNN
@@
 Wire Wire Line
 	1450 2550 1550 2550
+Connection ~ 1100 1750
+Wire Wire Line
+	1100 1750 1100 1700
+$Comp
+L KLIB_Connector_Prog:UART_01X03 J3
+U 1 1 5AD02C56
+P 4100 7000
+F 0 "J3" H 3921 7046 50  0000 R CNN
+F 1 "UART_01X03" H 3921 6955 50  0000 R CNN
+F 2 "Connector_PinHeader_2.54mm:PinHeader_1x03_P2.54mm_Vertical" H 4100 6600 50  0001 C CNN
+F 3 "~" H 4750 7200 50  0001 C CNN
+	1    4100 7000
+	-1   0    0    -1
+$EndComp
+$Comp
+L KLIB_Power:GND #PWR035
+U 1 1 5AD02C5D
+P 3800 7100
+F 0 "#PWR035" H 3800 6900 50  0001 C CNN
+F 1 "GND" H 3805 6927 50  0000 C CNN
+F 2 "" H 3800 7100 50  0001 C CNN
+F 3 "" H 3800 7100 50  0001 C CNN
+	1    3800 7100
+	-1   0    0    -1
+$EndComp
+Text Label 10900 4850 2    50   ~ 0
+DEBUG_UART_TX
+Text Label 10900 4950 2    50   ~ 0
+DEBUG_UART_RX
+Wire Wire Line
+	10150 4850 10900 4850
+Wire Wire Line
+	10150 4950 10900 4950
+Text Label 3050 6900 0    50   ~ 0
+DEBUG_UART_TX
+Text Label 3050 7000 0    50   ~ 0
+DEBUG_UART_RX
+Wire Wire Line
+	3800 6900 3050 6900
+Wire Wire Line
+	3800 7000 3050 7000
 Wire Bus Line
 	1650 6400 1650 7200
-Connection ~ 1100 1750
-Wire Wire Line
-	1100 1750 1100 1700
 $EndSCHEMATC
