File: hw/arm.sch (KiCad schematic (older format))
At the start: 13 parts, among them J3 UART_01X03, J4 SWD_01X04, U5 STM32F405RGTx

Commit message: updated schematic
Parts:
- added C18, C19, C20, C21: 12p, Capacitor_SMD:C_0805_2012Metric, symbol Device:C
- added Y1: ABM7-8.000MHZ-D2Y, Crystal:Crystal_SMD_2012-2Pin_2.0x1.2mm_HandSoldering, symbol Device:Crystal
- added Y2: IL3X2-HX5F12.5-32.768KHZ, Crystal:Crystal_SMD_2012-2Pin_2.0x1.2mm_HandSoldering, symbol Device:Crystal
Connections:
- net GND: now also C18.2, C19.2, C20.2, C21.2
- net OSC32_IN: now reaches U5.3 (PC14/RCC_OSC32_IN)
- net OSC32_IN: now also C20.1, Y2.1
- net OSC32_OUT: now reaches U5.4 (PC15/ADC1_EXTI15/ADC2_EXTI15/ADC3_EXTI15/RCC_OSC32_OUT)
- net OSC32_OUT: now also C21.1, Y2.2
- net OSC_IN: now reaches U5.5 (PH0/RCC_OSC_IN)
- net OSC_IN: now also C18.1, Y1.1
- net OSC_OUT: now reaches U5.6 (PH1/RCC_OSC_OUT)
- net OSC_OUT: now also C19.1, Y1.2
- no-connect marks 31 -> 27
Other:
- moved on the sheet: C10, C11
Changed lines of the file:
@@
 NoConn ~ 10150 4150
 NoConn ~ 10150 4050
-NoConn ~ 1550 5350
-NoConn ~ 1550 5250
 NoConn ~ 1550 5150
 NoConn ~ 1550 5050
@@
 NoConn ~ 1550 3850
 NoConn ~ 1550 3650
-NoConn ~ 1550 3450
-NoConn ~ 1550 3350
 $Comp
 L Device:C C10
 U 1 1 5AD22BDE
-P 750 2950
-F 0 "C10" H 865 2996 50  0000 L CNN
-F 1 "100n" H 865 2905 50  0000 L CNN
-F 2 "Capacitor_SMD:C_0805_2012Metric" H 788 2800 50  0001 C CNN
-F 3 "~" H 750 2950 50  0001 C CNN
-	1    750  2950
+P 750 2900
+F 0 "C10" H 865 2946 50  0000 L CNN
+F 1 "100n" H 865 2855 50  0000 L CNN
+F 2 "Capacitor_SMD:C_0805_2012Metric" H 788 2750 50  0001 C CNN
+F 3 "~" H 750 2900 50  0001 C CNN
+	1    750  2900
 	1    0    0    -1
 $EndComp
@@
 L Device:C C11
 U 1 1 5AD22C3E
-P 1250 2950
-F 0 "C11" H 1365 2996 50  0000 L CNN
-F 1 "100n" H 1365 2905 50  0000 L CNN
-F 2 "Capacitor_SMD:C_0805_2012Metric" H 1288 2800 50  0001 C CNN
-F 3 "~" H 1250 2950 50  0001 C CNN
-	1    1250 2950
+P 1250 2900
+F 0 "C11" H 1365 2946 50  0000 L CNN
+F 1 "100n" H 1365 2855 50  0000 L CNN
+F 2 "Capacitor_SMD:C_0805_2012Metric" H 1288 2750 50  0001 C CNN
+F 3 "~" H 1250 2900 50  0001 C CNN
+	1    1250 2900
 	1    0    0    -1
 $EndComp
@@
 L KLIB_Power:GND #PWR033
 U 1 1 5AD22D21
-P 1250 3100
-F 0 "#PWR033" H 1250 2900 50  0001 C CNN
-F 1 "GND" H 1255 2927 50  0000 C CNN
-F 2 "" H 1250 3100 50  0001 C CNN
-F 3 "" H 1250 3100 50  0001 C CNN
-	1    1250 3100
+P 1250 3050
+F 0 "#PWR033" H 1250 2850 50  0001 C CNN
+F 1 "GND" H 1255 2877 50  0000 C CNN
+F 2 "" H 1250 3050 50  0001 C CNN
+F 3 "" H 1250 3050 50  0001 C CNN
+	1    1250 3050
 	1    0    0    -1
 $EndComp
@@
 L KLIB_Power:GND #PWR031
 U 1 1 5AD22D74
-P 750 3100
-F 0 "#PWR031" H 750 2900 50  0001 C CNN
-F 1 "GND" H 755 2927 50  0000 C CNN
-F 2 "" H 750 3100 50  0001 C CNN
-F 3 "" H 750 3100 50  0001 C CNN
-	1    750  3100
-	1    0    0    -1
-$EndComp
-Wire Wire Line
-	750  2650 750  2800
+P 750 3050
+F 0 "#PWR031" H 750 2850 50  0001 C CNN
+F 1 "GND" H 755 2877 50  0000 C CNN
+F 2 "" H 750 3050 50  0001 C CNN
+F 3 "" H 750 3050 50  0001 C CNN
+	1    750  3050
+	1    0    0    -1
+$EndComp
+Wire Wire Line
+	750  2650 750  2750
 Wire Wire Line
 	1550 2750 1250 2750
-Wire Wire Line
-	1250 2750 1250 2800
 $Comp
 L Device:C C13
@@
 Wire Wire Line
 	3800 7000 3050 7000
+$Comp
+L Device:Crystal Y1
+U 1 1 5AD541EF
+P 2550 950
+F 0 "Y1" H 2550 1218 50  0000 C CNN
+F 1 "ABM7-8.000MHZ-D2Y" H 2550 1127 50  0000 C CNN
+F 2 "Crystal:Crystal_SMD_2012-2Pin_2.0x1.2mm_HandSoldering" H 2550 950 50  0001 C CNN
+F 3 "https://www.tme.eu/cz/details/abm7-8.000mhz-d2y/kremikove-rezonatory-smd/abracon/abm7-8000mhz-d2y-t/" H 2550 950 50  0001 C CNN
+	1    2550 950
+	1    0    0    -1
+$EndComp
+$Comp
+L Device:C C18
+U 1 1 5AD544FC
+P 2200 1150
+F 0 "C18" H 2315 1196 50  0000 L CNN
+F 1 "12p" H 2315 1105 50  0000 L CNN
+F 2 "Capacitor_SMD:C_0805_2012Metric" H 2238 1000 50  0001 C CNN
+F 3 "~" H 2200 1150 50  0001 C CNN
+	1    2200 1150
+	1    0    0    -1
+$EndComp
+$Comp
+L Device:C C19
+U 1 1 5AD545F5
+P 2900 1150
+F 0 "C19" H 3015 1196 50  0000 L CNN
+F 1 "12p" H 3015 1105 50  0000 L CNN
+F 2 "Capacitor_SMD:C_0805_2012Metric" H 2938 1000 50  0001 C CNN
+F 3 "~" H 2900 1150 50  0001 C CNN
+	1    2900 1150
+	1    0    0    -1
+$EndComp
+Wire Wire Line
+	2400 950  2200 950
+Wire Wire Line
+	2200 950  2200 1000
+Wire Wire Line
+	2700 950  2900 950
+Wire Wire Line
+	2900 950  2900 1000
+$Comp
+L KLIB_Power:GND #PWR040
+U 1 1 5AD597A8
+P 2200 1300
+F 0 "#PWR040" H 2200 1100 50  0001 C CNN
+F 1 "GND" H 2205 1127 50  0000 C CNN
+F 2 "" H 2200 1300 50  0001 C CNN
+F 3 "" H 2200 1300 50  0001 C CNN
+	1    2200 1300
+	1    0    0    -1
+$EndComp
+$Comp
+L KLIB_Power:GND #PWR041
+U 1 1 5AD597DA
+P 2900 1300
+F 0 "#PWR041" H 2900 1100 50  0001 C CNN
+F 1 "GND" H 2905 1127 50  0000 C CNN
+F 2 "" H 2900 1300 50  0001 C CNN
+F 3 "" H 2900 1300 50  0001 C CNN
+	1    2900 1300
+	1    0    0    -1
+$EndComp
+Text Label 1750 950  0    50   ~ 0
+OSC_IN
+Text Label 3350 950  2    50   ~ 0
+OSC_OUT
+Connection ~ 2200 950
+Wire Wire Line
+	1750 950  2200 950
+Wire Wire Line
+	2900 950  3350 950
+Connection ~ 2900 950
+$Comp
+L Device:Crystal Y2
+U 1 1 5AD6A6FE
+P 4350 950
+F 0 "Y2" H 4350 1218 50  0000 C CNN
+F 1 "IL3X2-HX5F12.5-32.768KHZ" H 4350 1127 50  0000 C CNN
+F 2 "Crystal:Crystal_SMD_2012-2Pin_2.0x1.2mm_HandSoldering" H 4350 950 50  0001 C CNN
+F 3 "https://www.tme.eu/cz/details/il3x2-hx5f-32.768k/kremikove-rezonatory-smd/ilsi/il3x2-hx5f125-32768khz/" H 4350 950 50  0001 C CNN
+	1    4350 950
+	1    0    0    -1
+$EndComp
+$Comp
+L Device:C C20
+U 1 1 5AD6A705
+P 4000 1150
+F 0 "C20" H 4115 1196 50  0000 L CNN
+F 1 "12p" H 4115 1105 50  0000 L CNN
+F 2 "Capacitor_SMD:C_0805_2012Metric" H 4038 1000 50  0001 C CNN
+F 3 "~" H 4000 1150 50  0001 C CNN
+	1    4000 1150
+	1    0    0    -1
+$EndComp
+$Comp
+L Device:C C21
+U 1 1 5AD6A70C
+P 4700 1150
+F 0 "C21" H 4815 1196 50  0000 L CNN
+F 1 "12p" H 4815 1105 50  0000 L CNN
+F 2 "Capacitor_SMD:C_0805_2012Metric" H 4738 1000 50  0001 C CNN
+F 3 "~" H 4700 1150 50  0001 C CNN
+	1    4700 1150
+	1    0    0    -1
+$EndComp
+Wire Wire Line
+	4200 950  4000 950
+Wire Wire Line
+	4000 950  4000 1000
+Wire Wire Line
+	4500 950  4700 950
+Wire Wire Line
+	4700 950  4700 1000
+$Comp
+L KLIB_Power:GND #PWR042
+U 1 1 5AD6A717
+P 4000 1300
+F 0 "#PWR042" H 4000 1100 50  0001 C CNN
+F 1 "GND" H 4005 1127 50  0000 C CNN
+F 2 "" H 4000 1300 50  0001 C CNN
+F 3 "" H 4000 1300 50  0001 C CNN
+	1    4000 1300
+	1    0    0    -1
+$EndComp
+$Comp
+L KLIB_Power:GND #PWR043
+U 1 1 5AD6A71D
+P 4700 1300
+F 0 "#PWR043" H 4700 1100 50  0001 C CNN
+F 1 "GND" H 4705 1127 50  0000 C CNN
+F 2 "" H 4700 1300 50  0001 C CNN
+F 3 "" H 4700 1300 50  0001 C CNN
+	1    4700 1300
+	1    0    0    -1
+$EndComp
+Text Label 3550 950  0    50   ~ 0
+OSC32_IN
+Text Label 5150 950  2    50   ~ 0
+OSC32_OUT
+Connection ~ 4000 950
+Wire Wire Line
+	3550 950  4000 950
+Wire Wire Line
+	4700 950  5150 950
+Connection ~ 4700 950
+Text Label 900  3350 0    50   ~ 0
+OSC_IN
+Text Label 900  3450 0    50   ~ 0
+OSC_OUT
+Text Label 900  5250 0    50   ~ 0
+OSC32_IN
+Text Label 900  5350 0    50   ~ 0
+OSC32_OUT
+Wire Wire Line
+	900  3350 1550 3350
+Wire Wire Line
+	900  3450 1550 3450
+Wire Wire Line
+	900  5250 1550 5250
+Wire Wire Line
+	900  5350 1550 5350
 Wire Bus Line
 	1650 6400 1650 7200

Commit message: created pcb
Connections:
- net ~RF_CONFIG: now also U5.15 (ADC1_IN1/ADC2_IN1/ADC3_IN1/TIM2_CH2/TIM5_CH2/UART4_RX/USART2_RTS/PA1); no longer U5.14 (ADC1_IN0/ADC2_IN0/ADC3_IN0/SYS_WKUP/TIM2_CH1/TIM2_ETR/TIM5_CH1/TIM8_ETR/UART4_TX/USART2_CTS/PA0)
- net ~RF_ENABLE: now also U5.14 (ADC1_IN0/ADC2_IN0/ADC3_IN0/SYS_WKUP/TIM2_CH1/TIM2_ETR/TIM5_CH1/TIM8_ETR/UART4_TX/USART2_CTS/PA0); no longer U5.15 (ADC1_IN1/ADC2_IN1/ADC3_IN1/TIM2_CH2/TIM5_CH2/UART4_RX/USART2_RTS/PA1)
Changed lines of the file:
@@
 Wire Wire Line
 	10150 2250 10400 2250
+Text HLabel 10400 2250 2    50   Output ~ 0
+~RF_CONFIG
 Text HLabel 10400 2150 2    50   Output ~ 0
-~RF_CONFIG
-Text HLabel 10400 2250 2    50   Output ~ 0
 ~RF_ENABLE
 Text Label 1200 2150 0    50   ~ 0
