File: hw/router.sch (KiCad schematic (older format))
At the start: 49 parts, among them J1 SMA, J2 USB_B, J3 SWD_01X04, J4 UART_01X03, U1 MCP1826S, U2 USBLC6-2SC6, U3 HM-TRP-869S, U4 CP2102, U5 STM32F401CEUx

Commit message: changed mcu from STM32F401CEUx to STM32F405RGTx and split schematic to more sheets
Parts:
- removed C10, C11, C12: 100n, symbol Device:C
- removed C13, C14: 1u, symbol Device:C
- removed C6: 4u7, symbol Device:C
- removed J3: SWD_01X04, Connector_PinHeader_2.54mm:PinHeader_1x04_P2.54mm_Vertical, symbol KLIB_Connector_Prog:SWD_01X04
- removed R3, R4: 10k, symbol Device:R
- removed U5: STM32F401CEUx, UFQFPN48, symbol MCU_ST_STM32:STM32F401CEUx
- added C8: 1u/50V, symbol Device:C
- C9: value 100n -> 1u/50V
- renumbered C7 to C6, C8 to C7, J2 to J1, J1 to J2, J4 to J3, R12 to R10, R5 to R3, R6 to R4, R7 to R5, R8 to R6, R9 to R7, R10 to R8, R11 to R9
Connections:
- net labels added: LED[7..0]
- net labels removed: DEBUG_UART_RX, DEBUG_UART_TX, SWCLK, SWDIO, ~RST
- wire segments 179 -> 109
- no-connect marks 23 -> 7
Other:
- moved on the sheet: C1, C2, C3, C4, C5, C6, C7, D1, D10, D2, D3, D4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

Commit message: updated schematic
Parts:
- removed J3: UART_01X03, Connector_PinHeader_2.54mm:PinHeader_1x03_P2.54mm_Vertical, symbol KLIB_Connector_Prog:UART_01X03
- C1, C5: value 1u -> 1u/50V; footprint (none) -> Capacitor_SMD:C_0805_2012Metric
- C2, C3, C4, C6, C7, C8, C9: footprint (none) -> Capacitor_SMD:C_0805_2012Metric
- D1: footprint (none) -> Diode_SMD:D_0603_1608Metric
- D10, D2, D3, D4, D5, D6, D7, D8, D9: footprint (none) -> LED_SMD:LED_0805_2012Metric
- J2: footprint (none) -> Connector_Coaxial:SMA_Jack_Vertical
- R1, R10, R2, R3, R4, R5, R6, R7, R8, R9: footprint (none) -> Resistor_SMD:R_0805_2012Metric
- U3: footprint (none) -> KLIB_RF_Module:HM-TRP-SMD
Connections:
- net +3V3: now also U3.1 (VCC)
- net GND: now also U3.3 (GND), U3.8 (GND)
- net at U3.9 (ANT): now also D1.1 (A1), J2.1 (In)
Other:
- moved on the sheet: C1, D1, J2
