File: hw/router.sch (KiCad schematic (older format))
At the start: 39 parts, among them J1 USB_B, J2 SMA, U1 MCP1826S, U2 USBLC6-2SC6, U3 HM-TRP-869S, U4 CP2102

Commit message: updated schematic
Parts:
- U4: footprint Housings_DFN_QFN:QFN-28-1EP_5x5mm_Pitch0.5mm -> Package_DFN_QFN:QFN-28-1EP_5x5mm_P0.5mm_EP3.35x3.35mm
Connections:
- net GND: now also U4.29 (GND), U4.3 (GND)
- net USB_UART_RTS: now also U4.23 (CTS); no longer U4.24 (RTS)
- net USB_UART_RX: now also U4.26 (TXD)
- net USB_UART_TX: now also U4.25 (RXD); no longer U4.26 (TXD)
- net USB_USRT_CTS: now also U4.24 (RTS); no longer U4.27 (DSR)
Changed lines of the file:
@@
-	1    0    0    -1
-$EndComp
-$Comp
-L KLIB_Interface:CP2102 U4
-U 1 1 5ABE9A5D
-P 4000 4200
-F 0 "U4" H 4200 5150 50  0000 L CNN
-F 1 "CP2102" H 4200 5050 50  0000 L CNN
-F 2 "Housings_DFN_QFN:QFN-28-1EP_5x5mm_Pitch0.5mm" H 4200 3250 50  0001 L CNN
-F 3 "https://www.silabs.com/documents/public/data-sheets/CP2102-9.pdf" H 4200 3150 50  0001 L CNN
-	1    4000 4200
 	1    0    0    -1
 $EndComp
@@
 L KLIB_Power:GND #PWR019
 U 1 1 5ABEB253
-P 4100 5200
-F 0 "#PWR019" H 4100 5000 50  0001 C CNN
-F 1 "GND" H 4105 5027 50  0000 C CNN
-F 2 "" H 4100 5200 50  0001 C CNN
-F 3 "" H 4100 5200 50  0001 C CNN
-	1    4100 5200
+P 4100 5100
+F 0 "#PWR019" H 4100 4900 50  0001 C CNN
+F 1 "GND" H 4105 4927 50  0000 C CNN
+F 2 "" H 4100 5100 50  0001 C CNN
+F 3 "" H 4100 5100 50  0001 C CNN
+	1    4100 5100
 	1    0    0    -1
 $EndComp
@@
 L KLIB_Power:GND #PWR017
 U 1 1 5ABEB288
-P 3900 5200
-F 0 "#PWR017" H 3900 5000 50  0001 C CNN
-F 1 "GND" H 3905 5027 50  0000 C CNN
-F 2 "" H 3900 5200 50  0001 C CNN
-F 3 "" H 3900 5200 50  0001 C CNN
-	1    3900 5200
+P 3900 5100
+F 0 "#PWR017" H 3900 4900 50  0001 C CNN
+F 1 "GND" H 3905 4927 50  0000 C CNN
+F 2 "" H 3900 5100 50  0001 C CNN
+F 3 "" H 3900 5100 50  0001 C CNN
+	1    3900 5100
 	1    0    0    -1
 $EndComp
@@
 Wire Wire Line
 	2950 3300 3250 3300
-Text Label 5200 3700 2    50   ~ 0
+Text Label 4650 3600 0    50   ~ 0
 USB_UART_TX
-Text Label 5200 3800 2    50   ~ 0
+Text Label 4650 3700 0    50   ~ 0
 USB_UART_RX
-Text Label 5200 4000 2    50   ~ 0
+Text Label 4650 3900 0    50   ~ 0
 USB_UART_RTS
-Text Label 5200 4100 2    50   ~ 0
+Text Label 4650 4000 0    50   ~ 0
 USB_USRT_CTS
-NoConn ~ 4600 4800
+NoConn ~ 4600 4100
 NoConn ~ 4600 4700
-NoConn ~ 4600 4500
+NoConn ~ 4600 4600
 NoConn ~ 4600 4400
 NoConn ~ 4600 4300
@@
 	4150 1700 6800 1700
 Wire Wire Line
-	5250 3700 5250 2200
-Wire Wire Line
-	4600 3700 5250 3700
-Wire Wire Line
-	5350 3800 5350 2300
-Wire Wire Line
-	4600 3800 5350 3800
-Wire Wire Line
 	6800 2200 5250 2200
 Wire Wire Line
 	6800 2300 5350 2300
 Wire Wire Line
-	5450 4000 5450 2400
-Wire Wire Line
 	5450 2400 6800 2400
 Wire Wire Line
-	4600 4000 5450 4000
-Wire Wire Line
-	5550 4100 5550 2500
-Wire Wire Line
 	5550 2500 6800 2500
-Wire Wire Line
-	4600 4100 5550 4100
 Entry Wire Line
 	7450 4450 7550 4550
@@
 	2600 1800 1900 1800
 Connection ~ 1900 1800
+Wire Wire Line
+	4600 3600 5250 3600
+Wire Wire Line
+	5250 3600 5250 2200
+Wire Wire Line
+	4600 3900 5450 3900
+Wire Wire Line
+	5450 3900 5450 2400
+Wire Wire Line
+	5550 4000 5550 2500
+Wire Wire Line
+	4600 4000 5550 4000
+Wire Wire Line
+	5350 3700 5350 2300
+Wire Wire Line
+	4600 3700 5350 3700
 Wire Bus Line
 	7450 3400 7450 5150
+$Comp
+L KLIB_Interface:CP2102 U4
+U 1 1 5AD4FD61
+P 4000 4200
+F 0 "U4" H 4200 5150 50  0000 L CNN
+F 1 "CP2102" H 4200 5050 50  0000 L CNN
+F 2 "Package_DFN_QFN:QFN-28-1EP_5x5mm_P0.5mm_EP3.35x3.35mm" H 4200 3350 50  0001 L CNN
+F 3 "https://www.silabs.com/documents/public/data-sheets/CP2102-9.pdf" H 4200 3150 50  0001 L CNN
+	1    4000 4200
+	1    0    0    -1
+$EndComp
 $EndSCHEMATC

Commit message: added placement file
Parts:
- J1: symbol Connector_Specialized:USB_B -> Connector:USB_B
- J2: symbol Connector_Specialized:Conn_Coaxial -> Connector:Conn_Coaxial
Other:
- moved on the sheet: J2
Changed lines of the file:
@@
 $EndComp
 $Comp
-L Connector_Specialized:USB_B J1
+L Connector:USB_B J1
 U 1 1 5ABE9679
 P 1200 4200
@@
 $EndComp
 $Comp
-L Connector_Specialized:Conn_Coaxial J2
+L Connector:Conn_Coaxial J2
 U 1 1 5ABFBD92
 P 1650 1800
@@
 Wire Wire Line
 	1650 2300 1650 2000
-Wire Wire Line
-	1800 1800 1900 1800
 $Comp
 L Device:D_TVS D1
@@
 Wire Wire Line
 	2600 1800 1900 1800
-Connection ~ 1900 1800
 Wire Wire Line
 	4600 3600 5250 3600
@@
 Wire Wire Line
 	4600 3700 5350 3700
-Wire Bus Line
-	7450 3400 7450 5150
 $Comp
 L KLIB_Interface:CP2102 U4
@@
 	1    0    0    -1
 $EndComp
+Wire Wire Line
+	1850 1800 1900 1800
+Wire Bus Line
+	7450 3400 7450 5150
+Connection ~ 1900 1800
 $EndSCHEMATC
